Commit message: Modifing robot to incorporate grippers, changing front of the robot to the other side as the other way was not correct

File: malakrobo_description/urdf/malakrobo2.xacro (robot description, xacro)
@@ -80,44 +80,44 @@
 </link>
 <link name="left_fence">
-  <visual>
-    <origin rpy="1.0 1.57 1.57" xyz="0 0 0"/>
-    <geometry>
-      <box size="0.1 0.01 0.12"/>
-    </geometry>
-  </visual>
-  <collision>
-    <origin rpy="1.57 -1.0 1.57" xyz="0 0 0"/>
-    <geometry>
-      <box size="0.1 0.01 0.12"/>
-    </geometry>
-  </collision>
-  <inertial>
-    <mass value="1"/>
-    <origin rpy="0 0 0" xyz="0 0 0"/>
-    <inertia ixx="1" ixy="0" ixz="0" iyy="1" iyz="0" izz="1"/>
-  </inertial>
+<visual>
+  <origin rpy="1.57 -1.0 1.57" xyz="0 0 0"/>
+  <geometry>
+    <box size="0.1 0.01 0.12"/>
+  </geometry>
+</visual>
+<collision>
+  <origin rpy="1.57 -1.0 1.57" xyz="0 0 0"/>
+  <geometry>
+    <box size="0.1 0.01 0.12"/>
+  </geometry>
+</collision>
+<inertial>
+  <mass value="1"/>
+  <origin rpy="0 0 0" xyz="0 0 0"/>
+  <inertia ixx="1" ixy="0" ixz="0" iyy="1" iyz="0" izz="1"/>
+</inertial>
 </link>
 <link name="right_fence">
-  <visual>
-    <origin rpy="-1.0 1.57 1.57" xyz="0 0 0"/>
-    <geometry>
-      <box size="0.1 0.01 0.12"/>
-    </geometry>
-  </visual>
-  <collision>
-    <origin rpy="1.57 1.0 1.57" xyz="0 0 0"/>
-    <geometry>
-      <box size="0.1 0.01 0.12"/>
-    </geometry>
-  </collision>
-  <inertial>
-    <mass value="1"/>
-    <origin rpy="0 0 0" xyz="0 0 0"/>
-    <inertia ixx="1" ixy="0" ixz="0" iyy="1" iyz="0" izz="1"/>
-  </inertial>
+<visual>
+  <origin rpy="1.57 1.0 1.57" xyz="0 0 0"/>
+  <geometry>
+    <box size="0.1 0.01 0.12"/>
+  </geometry>
+</visual>
+<collision>
+  <origin rpy="1.57 1.0 1.57" xyz="0 0 0"/>
+  <geometry>
+    <box size="0.1 0.01 0.12"/>
+  </geometry>
+</collision>
+<inertial>
+  <mass value="1"/>
+  <origin rpy="0 0 0" xyz="0 0 0"/>
+  <inertia ixx="1" ixy="0" ixz="0" iyy="1" iyz="0" izz="1"/>
+</inertial>
 </link>
 <link name="left_fence_front">
 <visual>
-<origin rpy="1.50 1.57 1.57" xyz="0 0 0"/>
+<origin rpy="1.57 -1.5 1.57" xyz="0 0 0"/>
 <geometry>
   <box size="0.1 0.01 0.075"/>
@@ -138,5 +138,5 @@
 <link name="right_fence_front">
 <visual>
-<origin rpy="-1.5 1.57 1.57" xyz="0 0 0"/>
+<origin rpy="1.57 1.5 1.57" xyz="0 0 0"/>
 <geometry>
   <box size="0.1 0.01 0.075"/>
