Commit message: Redesigning the robot

File: malakrobo_description/urdf/malakrobo.xacro (robot description, xacro)
@@ -7,17 +7,37 @@
     <origin rpy="0 0 0" xyz="0 0 0.1"/>
     <geometry>
-      <box size="0.1 0.1 0.1"/>
-    </geometry>
-    <material name="silver"/>
-  </visual>
-  <collision>
-    <origin rpy="0 0 0" xyz="0 0 0.1"/>
-    <geometry>
-      <box size="0.1 0.1 0.1"/>
-    </geometry>
-  </collision>
-  <inertial>
-    <mass value="0.5"/>
-    <origin xyz="0 0 0.1" rpy="0 0 0"/>
+      <cylinder radius="0.2" length="0.02"/>
+    </geometry>
+    <material name="silver"/>
+  </visual>
+  <collision>
+    <origin rpy="0 0 0" xyz="0 0 0.1"/>
+    <geometry>
+      <cylinder radius="0.2" length="0.02"/>
+    </geometry>
+  </collision>
+  <inertial>
+    <mass value="75"/>
+    <origin rpy="0 0 0" xyz="0 0 0"/>
+    <inertia ixx="1" ixy="0" ixz="0" iyy="1" iyz="0" izz="1"/>
+  </inertial>
+</link>
+<link name="base2">
+  <visual>
+    <origin rpy="0 0 0" xyz="0 0 0.1"/>
+    <geometry>
+      <box size="0.1 0.4 0.02"/>
+    </geometry>
+    <material name="silver"/>
+  </visual>
+  <collision>
+    <origin rpy="0 0 0" xyz="0 0 0.1"/>
+    <geometry>
+      <box size="0.1 0.4 0.02"/>
+    </geometry>
+  </collision>
+  <inertial>
+    <mass value="75"/>
+    <origin rpy="0 0 0" xyz="0 0 0"/>
     <inertia ixx="1" ixy="0" ixz="0" iyy="1" iyz="0" izz="1"/>
   </inertial>
@@ -25,19 +45,19 @@
 <link name="left_wheel">
   <visual>
-    <origin rpy="1.57079633 0 0" xyz="0 0 0"/>
-    <geometry>
-      <cylinder radius="0.1" length="0.05"/>
-    </geometry>
-    <material name="rubber"/>
-  </visual>
-  <collision>
-    <origin rpy="1.57079633 0 0" xyz="0 0 0"/>
-    <geometry>
-      <cylinder radius="0.1" length="0.05"/>
-    </geometry>
-  </collision>
-  <inertial>
-    <mass value="0.1"/>
-    <origin rpy="1.57079633 0 0" xyz="0 0 0"/>
+    <origin rpy="1.57 0 0" xyz="0 0 0"/>
+    <geometry>
+      <cylinder radius="0.1" length="0.05"/>
+    </geometry>
+    <material name="silver"/>
+  </visual>
+  <collision>
+    <origin rpy="1.57 0 0" xyz="0 0 0"/>
+    <geometry>
+      <cylinder radius="0.1" length="0.05"/>
+    </geometry>
+  </collision>
+  <inertial>
+    <mass value="0.5"/>
+    <origin rpy="0 0 0" xyz="0 0 0"/>
     <inertia ixx="1" ixy="0" ixz="0" iyy="1" iyz="0" izz="1"/>
   </inertial>
@@ -45,31 +65,145 @@
 <link name="right_wheel">
   <visual>
-    <origin rpy="-1.57079633 0 0" xyz="0 0 0"/>
-    <geometry>
-      <cylinder radius="0.1" length="0.05"/>
-    </geometry>
-    <material name="rubber"/>
-  </visual>
-  <collision>
-    <origin rpy="-1.57079633 0 0" xyz="0 0 0"/>
-    <geometry>
-      <cylinder radius="0.1" length="0.05"/>
-    </geometry>
-  </collision>
-  <inertial>
-    <mass value="0.1"/>
-    <origin rpy="-1.57079633 0 0" xyz="0 0 0"/>
-    <inertia ixx="1" ixy="0" ixz="0" iyy="1" iyz="0" izz="1"/>
-  </inertial>
-</link>
+    <origin rpy="1.57 0 0" xyz="0 0 0"/>
+    <geometry>
+      <cylinder radius="0.1" length="0.05"/>
+    </geometry>
+    <material name="silver"/>
+  </visual>
+  <collision>
+    <origin rpy="1.57 0 0" xyz="0 0 0"/>
+    <geometry>
+      <cylinder radius="0.1" length="0.05"/>
+    </geometry>
+  </collision>
+  <inertial>
+    <mass value="0.5"/>
+    <origin rpy="0 0 0" xyz="0 0 0"/>
+    <inertia ixx="1" ixy="0" ixz="0" iyy="1" iyz="0" izz="1"/>
+  </inertial>
+</link>
+<link name="balance_wheel_mount_back">
+  <visual>
+    <origin rpy="0 0 0" xyz="0 0 0"/>
+    <geometry>
+      <box size="0.05 0.05 0.08"/>
+    </geometry>
+    <material name="silver"/>
+  </visual>
+  <collision>
+    <origin rpy="0 0 0" xyz="0 0 0"/>
+    <geometry>
+      <box size="0.05 0.05 0.08"/>
+    </geometry>
+  </collision>
+  <inertial>
+    <mass value="0.5"/>
+    <origin rpy="0 0 0" xyz="0 0 0"/>
+    <inertia ixx="1" ixy="0" ixz="0" iyy="1" iyz="0" izz="1"/>
+  </inertial>
+</link>
+<link name="balance_wheel_mount_front">
+  <visual>
+    <origin rpy="0 0 0" xyz="0 0 0"/>
+    <geometry>
+      <box size="0.05 0.05 0.08"/>
+    </geometry>
+    <material name="silver"/>
+  </visual>
+  <collision>
+    <origin rpy="0 0 0" xyz="0 0 0"/>
+    <geometry>
+      <box size="0.05 0.05 0.08"/>
+    </geometry>
+  </collision>
+  <inertial>
+    <mass value="0.5"/>
+    <origin rpy="0 0 0" xyz="0 0 0"/>
+    <inertia ixx="1" ixy="0" ixz="0" iyy="1" iyz="0" izz="1"/>
+  </inertial>
+</link>
+<link name="balance_ball_front">
+  <visual>
+    <origin rpy="0 0 0" xyz="0 0 0"/>
+    <geometry>
+      <sphere radius="0.025"/>
+    </geometry>
+    <material name="silver"/>
+  </visual>
+  <collision>
+    <origin rpy="0 0 0" xyz="0 0 0"/>
+    <geometry>
+      <sphere radius="0.025"/>
+    </geometry>
+  </collision>
+  <inertial>
+    <mass value="0.5"/>
+    <origin rpy="0 0 0" xyz="0 0 0"/>
+    <inertia ixx="0.001" ixy="0.0" ixz="0.0"
+               iyy="0.001" iyz="0.0"
+               izz="0.001" />
+  </inertial>
+</link>
+<link name="balance_ball_back">
+  <visual>
+    <origin rpy="0 0 0" xyz="0 0 0"/>
+    <geometry>
+      <sphere radius="0.025"/>
+    </geometry>
+    <material name="silver"/>
+  </visual>
+  <collision>
+    <origin rpy="0 0 0" xyz="0 0 0"/>
+    <geometry>
+      <sphere radius="0.025"/>
+    </geometry>
+  </collision>
+  <inertial>
+    <mass value="0.5"/>
+    <origin rpy="0 0 0" xyz="0 0 0"/>
+    <inertia ixx="0.001" ixy="0.0" ixz="0.0"
+               iyy="0.001" iyz="0.0"
+               izz="0.001" />
+  </inertial>
+</link>
+<joint name="base_joint" type="fixed">
+  <origin rpy="0 0 0" xyz="0 0 0"/>
+  <parent link="base_link"/>
+  <child link="base2"/>
+  <axis xyz="0.0 1.0 0.0"/>
+</joint>
+<joint name="base_balance_back" type="fixed">
+  <origin rpy="0 0 0" xyz="0.15 0 0.05"/>
+  <parent link="base2"/>
+  <child link="balance_wheel_mount_back"/>
+  <axis xyz="0.0 1.0 0.0"/>
+</joint>
+<joint name="base_balance_front" type="fixed">
+  <origin rpy="0 0 0" xyz="-0.15 0 0.05"/>
+  <parent link="base2"/>
+  <child link="balance_wheel_mount_front"/>
+  <axis xyz="0.0 1.0 0.0"/>
+</joint>
+<joint name="balance_ball_front" type="continuous">
+  <origin rpy="0 0 0" xyz="0 0 -0.03"/>
+  <parent link="balance_wheel_mount_front"/>
+  <child link="balance_ball_front"/>
+  <axis xyz="0.0 1.0 0.0"/>
+</joint>
+<joint name="balance_ball_back" type="continuous">
+  <origin rpy="0 0 0" xyz="0 0 -0.03"/>
+  <parent link="balance_wheel_mount_back"/>
+  <child link="balance_ball_back"/>
+  <axis xyz="0.0 1.0 0.0"/>
+</joint>
 <joint name="base_to_left_wheel" type="continuous">
-  <origin rpy="0 0 0" xyz="0 -0.075 0.1"/>
-  <parent link="base_link"/>
+  <origin rpy="0 0 0" xyz="0 -0.225 0.1"/>
+  <parent link="base2"/>
   <child link="left_wheel"/>
   <axis xyz="0.0 1.0 0.0"/>
 </joint>
 <joint name="base_to_right_wheel" type="continuous">
-  <origin rpy="0 0 0" xyz="0 0.075 0.1"/>
-  <parent link="base_link"/>
+  <origin rpy="0 0 0" xyz="0 0.225 0.1"/>
+  <parent link="base2"/>
   <child link="right_wheel"/>
   <axis xyz="0.0 1.0 0.0"/>

Commit message: Adding camera and laser

File: malakrobo_description/urdf/malakrobo.xacro (robot description, xacro)
@@ -1,56 +1,134 @@
 <?xml version="1.0" ?>
 <robot name="malakrobo" xmlns:xacro="http://www.ros.org/wiki/xacro">
-<xacro:include filename="$(find malakrobo_description)/urdf/materials.xacro" />
-<xacro:include filename="$(find malakrobo_description)/urdf/malakrobo.gazebo" />
-<link name="base_link">
+  <xacro:property name="cameraSize" value="0.05"/>
+  <xacro:property name="cameraMass" value="0.1"/>
+  <xacro:include filename="$(find malakrobo_description)/urdf/materials.xacro" />
+  <xacro:include filename="$(find malakrobo_description)/urdf/malakrobo.gazebo" />
+  <link name="base_link">
+    <visual>
+      <origin rpy="0 0 0" xyz="0 0 0.1"/>
+      <geometry>
+        <cylinder radius="0.2" length="0.02"/>
+      </geometry>
+    </visual>
+    <collision>
+      <origin rpy="0 0 0" xyz="0 0 0.1"/>
+      <geometry>
+        <cylinder radius="0.2" length="0.02"/>
+      </geometry>
+    </collision>
+    <inertial>
+      <mass value="5"/>
+      <origin rpy="0 0 0" xyz="0 0 0"/>
+      <inertia ixx="1" ixy="0" ixz="0" iyy="1" iyz="0" izz="1"/>
+    </inertial>
+  </link>
+  <link name="base2">
+    <visual>
+      <origin rpy="0 0 0" xyz="0 0 0.1"/>
+      <geometry>
+        <box size="0.1 0.4 0.02"/>
+      </geometry>
+    </visual>
+    <collision>
+      <origin rpy="0 0 0" xyz="0 0 0.1"/>
+      <geometry>
+        <box size="0.1 0.4 0.02"/>
+      </geometry>
+    </collision>
+    <inertial>
+      <mass value="5"/>
+      <origin rpy="0 0 0" xyz="0 0 0"/>
+      <inertia ixx="1" ixy="0" ixz="0" iyy="1" iyz="0" izz="1"/>
+    </inertial>
+  </link>
+  <link name="base3">
+    <visual>
+      <origin rpy="0 0 0" xyz="0 0 0.1"/>
+      <geometry>
+        <box size="0.15 0.25 0.02"/>
+      </geometry>
+    </visual>
+    <collision>
+      <origin rpy="0 0 0" xyz="0 0 0.1"/>
+      <geometry>
+        <box size="0.15 0.25 0.02"/>
+      </geometry>
+    </collision>
+    <inertial>
+      <mass value="1"/>
+      <origin rpy="0 0 0" xyz="0 0 0"/>
+      <inertia ixx="1" ixy="0" ixz="0" iyy="1" iyz="0" izz="1"/>
+    </inertial>
+  </link>
+  <link name="base_fence">
+    <visual>
+      <origin rpy="0 0 0" xyz="0 0 0.1"/>
+      <geometry>
+        <box size="0.02 0.25 0.1"/>
+      </geometry>
+    </visual>
+    <collision>
+      <origin rpy="0 0 0" xyz="0 0 0.1"/>
+      <geometry>
+        <box size="0.02 0.25 0.1"/>
+      </geometry>
+    </collision>
+    <inertial>
+      <mass value="1"/>
+      <origin rpy="0 0 0" xyz="0 0 0"/>
+      <inertia ixx="1" ixy="0" ixz="0" iyy="1" iyz="0" izz="1"/>
+    </inertial>
+  </link>
+  <link name="left_fence">
+    <visual>
+      <origin rpy="1.0 1.57 1.57" xyz="0 0 0"/>
+      <geometry>
+        <box size="0.1 0.01 0.12"/>
+      </geometry>
+    </visual>
+    <collision>
+      <origin rpy="1.57 -1.0 1.57" xyz="0 0 0"/>
+      <geometry>
+        <box size="0.1 0.01 0.12"/>
+      </geometry>
+    </collision>
+    <inertial>
+      <mass value="1"/>
+      <origin rpy="0 0 0" xyz="0 0 0"/>
+      <inertia ixx="1" ixy="0" ixz="0" iyy="1" iyz="0" izz="1"/>
+    </inertial>
+  </link>
+  <link name="right_fence">
+    <visual>
+      <origin rpy="-1.0 1.57 1.57" xyz="0 0 0"/>
+      <geometry>
+        <box size="0.1 0.01 0.12"/>
+      </geometry>
+    </visual>
+    <collision>
+      <origin rpy="1.57 1.0 1.57" xyz="0 0 0"/>
+      <geometry>
+        <box size="0.1 0.01 0.12"/>
+      </geometry>
+    </collision>
+    <inertial>
+      <mass value="1"/>
+      <origin rpy="0 0 0" xyz="0 0 0"/>
+      <inertia ixx="1" ixy="0" ixz="0" iyy="1" iyz="0" izz="1"/>
+    </inertial>
+  </link>
+  <link name="left_fence_front">
   <visual>
-    <origin rpy="0 0 0" xyz="0 0 0.1"/>
-    <geometry>
-      <cylinder radius="0.2" length="0.02"/>
-    </geometry>
+  <origin rpy="1.5 1.57 1.57" xyz="0 0 0"/>
+  <geometry>
+    <box size="0.1 0.01 0.075"/>
+  </geometry>
   </visual>
   <collision>
-    <origin rpy="0 0 0" xyz="0 0 0.1"/>
-    <geometry>
-      <cylinder radius="0.2" length="0.02"/>
-    </geometry>
-  </collision>
-  <inertial>
-    <mass value="5"/>
-    <origin rpy="0 0 0" xyz="0 0 0"/>
-    <inertia ixx="1" ixy="0" ixz="0" iyy="1" iyz="0" izz="1"/>
-  </inertial>
-</link>
-<link name="base2">
-  <visual>
-    <origin rpy="0 0 0" xyz="0 0 0.1"/>
-    <geometry>
-      <box size="0.1 0.4 0.02"/>
-    </geometry>
-  </visual>
-  <collision>
-    <origin rpy="0 0 0" xyz="0 0 0.1"/>
-    <geometry>
-      <box size="0.1 0.4 0.02"/>
-    </geometry>
-  </collision>
-  <inertial>
-    <mass value="5"/>
-    <origin rpy="0 0 0" xyz="0 0 0"/>
-    <inertia ixx="1" ixy="0" ixz="0" iyy="1" iyz="0" izz="1"/>
-  </inertial>
-</link>
-<link name="base3">
-  <visual>
-    <origin rpy="0 0 0" xyz="0 0 0.1"/>
-    <geometry>
-      <box size="0.15 0.25 0.02"/>
-    </geometry>
-  </visual>
-  <collision>
-    <origin rpy="0 0 0" xyz="0 0 0.1"/>
-    <geometry>
-      <box size="0.15 0.25 0.02"/>
-    </geometry>
+  <origin rpy="1.57 -1.5 1.57" xyz="0 0 0"/>
+  <geometry>
+    <box size="0.1 0.01 0.075"/>
+  </geometry>
   </collision>
   <inertial>
@@ -59,17 +137,17 @@
     <inertia ixx="1" ixy="0" ixz="0" iyy="1" iyz="0" izz="1"/>
   </inertial>
-</link>
-<link name="base_fence">
+  </link>
+  <link name="right_fence_front">
   <visual>
-    <origin rpy="0 0 0" xyz="0 0 0.1"/>
-    <geometry>
-      <box size="0.02 0.25 0.1"/>
-    </geometry>
+  <origin rpy="-1.5 1.57 1.57" xyz="0 0 0"/>
+  <geometry>
+    <box size="0.1 0.01 0.075"/>
+  </geometry>
   </visual>
   <collision>
-    <origin rpy="0 0 0" xyz="0 0 0.1"/>
-    <geometry>
-      <box size="0.02 0.25 0.1"/>
-    </geometry>
+  <origin rpy="1.57 1.5 1.57" xyz="0 0 0"/>
+  <geometry>
+    <box size="0.1 0.01 0.075"/>
+  </geometry>
   </collision>
   <inertial>
@@ -78,342 +156,319 @@
     <inertia ixx="1" ixy="0" ixz="0" iyy="1" iyz="0" izz="1"/>
   </inertial>
-</link>
-<link name="left_fence">
-  <visual>
-    <origin rpy="1.0 1.57 1.57" xyz="0 0 0"/>
-    <geometry>
-      <box size="0.1 0.01 0.12"/>
-    </geometry>
-  </visual>
-  <collision>
-    <origin rpy="1.57 -1.0 1.57" xyz="0 0 0"/>
-    <geometry>
-      <box size="0.1 0.01 0.12"/>
-    </geometry>
-  </collision>
-  <inertial>
-    <mass value="1"/>
+  </link>
+  <link name="front_caster_base">
+    <visual>
+      <origin rpy="0 0 0" xyz="0 0 0"/>
+      <geometry>
+        <box size="0.075 0.075 0.02"/>
+      </geometry>
+    </visual>
+    <collision>
+      <origin rpy="0 0 0" xyz="0 0 0"/>
+      <geometry>
+        <box size="0.075 0.075 0.02"/>
+      </geometry>
+    </collision>
+    <inertial>
+      <mass value="0.5"/>
+      <origin rpy="0 0 0" xyz="0 0 0"/>
+      <inertia ixx="1" ixy="0" ixz="0" iyy="1" iyz="0" izz="1"/>
+    </inertial>
+  </link>
+  <link name="back_caster_base">
+    <visual>
+      <origin rpy="0 0 0" xyz="0 0 0"/>
+      <geometry>
+        <box size="0.075 0.075 0.02"/>
+      </geometry>
+    </visual>
+    <collision>
+      <origin rpy="0 0 0" xyz="0 0 0"/>
+      <geometry>
+        <box size="0.075 0.075 0.02"/>
+      </geometry>
+    </collision>
+    <inertial>
+      <mass value="0.5"/>
+      <origin rpy="0 0 0" xyz="0 0 0"/>
+      <inertia ixx="1" ixy="0" ixz="0" iyy="1" iyz="0" izz="1"/>
+    </inertial>
+  </link>
+  <link name="front_caster_side">
+    <visual>
+      <origin rpy="0 0 0" xyz="0 0 0"/>
+      <geometry>
+        <box size="0.075 0.02 0.05"/>
+      </geometry>
+    </visual>
+    <collision>
+      <origin rpy="0 0 0" xyz="0 0 0"/>
+      <geometry>
+        <box size="0.075 0.02 0.05"/>
+      </geometry>
+    </collision>
+    <inertial>
+      <mass value="0.5"/>
+      <origin rpy="0 0 0" xyz="0 0 0"/>
+      <inertia ixx="1" ixy="0" ixz="0" iyy="1" iyz="0" izz="1"/>
+    </inertial>
+  </link>
+  <link name="back_caster_side">
+    <visual>
+      <origin rpy="0 0 0" xyz="0 0 0"/>
+      <geometry>
+        <box size="0.075 0.02 0.05"/>
+      </geometry>
+    </visual>
+    <collision>
+      <origin rpy="0 0 0" xyz="0 0 0"/>
+      <geometry>
+        <box size="0.075 0.02 0.05"/>
+      </geometry>
+    </collision>
+    <inertial>
+      <mass value="0.5"/>
+      <origin rpy="0 0 0" xyz="0 0 0"/>
+      <inertia ixx="1" ixy="0" ixz="0" iyy="1" iyz="0" izz="1"/>
+    </inertial>
+  </link>
+  <link name="front_caster_wheel">
+    <visual>
+      <origin rpy="1.57 0 0" xyz="0 0 0"/>
+      <geometry>
+        <cylinder radius="0.03" length="0.035"/>
+      </geometry>
+    </visual>
+    <collision>
+      <origin rpy="1.57 0 0" xyz="0 0 0"/>
+      <geometry>
+        <cylinder radius="0.03" length="0.035"/>
+      </geometry>
+    </collision>
+    <inertial>
+      <mass value="5"/>
+      <origin rpy="0 0 0" xyz="0 0 0"/>
+      <inertia ixx="1" ixy="0" ixz="0" iyy="1" iyz="0" izz="1"/>
+    </inertial>
+  </link>
+  <link name="back_caster_wheel">
+    <visual>
+      <origin rpy="-1.57 0 0" xyz="0 0 0"/>
+      <geometry>
+        <cylinder radius="0.03" length="0.035"/>
+      </geometry>
+    </visual>
+    <collision>
+      <origin rpy="-1.57 0 0" xyz="0 0 0"/>
+      <geometry>
+        <cylinder radius="0.03" length="0.035"/>
+      </geometry>
+    </collision>
+    <inertial>
+      <mass value="5"/>
+      <origin rpy="0 0 0" xyz="0 0 0"/>
+      <inertia ixx="1" ixy="0" ixz="0" iyy="1" iyz="0" izz="1"/>
+    </inertial>
+  </link>
+  <link name="left_wheel">
+    <visual>
+      <origin rpy="1.57 0 0" xyz="0 0 0"/>
+      <geometry>
+        <cylinder radius="0.1" length="0.05"/>
+      </geometry>
+    </visual>
+    <collision>
+      <origin rpy="1.57 0 0" xyz="0 0 0"/>
+      <geometry>
+        <cylinder radius="0.1" length="0.05"/>
+      </geometry>
+    </collision>
+    <inertial>
+      <mass value="5"/>
+      <origin rpy="0 0 0" xyz="0 0 0"/>
+      <inertia ixx="1" ixy="0" ixz="0" iyy="1" iyz="0" izz="1"/>
+    </inertial>
+  </link>
+  <link name="right_wheel">
+    <visual>
+      <origin rpy="1.57 0 0" xyz="0 0 0"/>
+      <geometry>
+        <cylinder radius="0.1" length="0.05"/>
+      </geometry>
+    </visual>
+    <collision>
+      <origin rpy="1.57 0 0" xyz="0 0 0"/>
+      <geometry>
+        <cylinder radius="0.1" length="0.05"/>
+      </geometry>
+    </collision>
+    <inertial>
+      <mass value="5"/>
+      <origin rpy="0 0 0" xyz="0 0 0"/>
+      <inertia ixx="1" ixy="0" ixz="0" iyy="1" iyz="0" izz="1"/>
+    </inertial>
+  </link>
+  <link name="camera">
+    <collision>
+      <origin xyz="0 0 0" rpy="0 0 0"/>
+      <geometry>
+        <box size="${cameraSize} ${cameraSize} ${cameraSize}"/>
+      </geometry>
+    </collision>
+    <visual>
+      <origin xyz="0 0 0" rpy="0 0 0"/>
+      <geometry>
+        <box size="${cameraSize} ${cameraSize} ${cameraSize}"/>
+      </geometry>
+      <material name="green"/>
+    </visual>
+    <inertial>
+      <mass value="${cameraMass}" />
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
Commit message: Updating sensor config (disabled GPU for it to work)

File: malakrobo_description/urdf/malakrobo.xacro (robot description, xacro)
@@ -309,4 +309,23 @@
     </inertial>
   </link>
+  <link name="sensor_base">
+    <collision>
+      <origin xyz="0 0 0" rpy="0 0 0"/>
+      <geometry>
+        <box size="0.1 0.1 0.2"/>
+      </geometry>
+    </collision>
+    <visual>
+      <origin xyz="0 0 0" rpy="0 0 0"/>
+      <geometry>
+        <box size="0.05 0.05 0.2"/>
+      </geometry>
+    </visual>
+    <inertial>
+      <mass value="1e-5" />
+      <origin xyz="0 0 0" rpy="0 0 0"/>
+      <inertia ixx="1e-6" ixy="0" ixz="0" iyy="1e-6" iyz="0" izz="1e-6" />
+    </inertial>
+  </link>
   <link name="camera">
     <collision>
@@ -335,5 +354,5 @@
       <origin xyz="0 0 0" rpy="0 0 0"/>
       <geometry>
-    <box size="0.1 0.1 0.1"/>
+        <box size="0.1 0.1 0.1"/>
       </geometry>
     </collision>
@@ -350,14 +369,20 @@
     </inertial>
   </link>
+  <joint name="sensor_base_joint" type="fixed">
+    <axis xyz="0 0 0" />
+    <origin xyz="-0.15 0 0.20" rpy="0 0 0"/>
+    <parent link="base_link"/>
+    <child link="sensor_base"/>
+  </joint>
   <joint name="camera_joint" type="fixed">
     <axis xyz="0 0 0" />
-    <origin xyz="-0.025 0 0.1" rpy="0 0 3.14"/>
-    <parent link="base_fence"/>
+    <origin xyz="-0.025 0 0.05" rpy="0 0 3.14"/>
+    <parent link="sensor_base"/>
     <child link="camera"/>
   </joint>
   <joint name="hokuyo_joint" type="fixed">
     <axis xyz="0 1 0" />
-    <origin xyz="0 0 0.45" rpy="0 0 3.14"/>
-    <parent link="base_link"/>
+    <origin xyz="0 0 0.13" rpy="0 0 3.14"/>
+    <parent link="sensor_base"/>
     <child link="hokuyo"/>
   </joint>

File: malakrobo_description/urdf/malakrobo2.xacro (robot description, xacro)
@@ -80,40 +80,40 @@
 </link>
 <link name="left_fence">
-<visual>
-  <origin rpy="1.57 -1.0 1.57" xyz="0 0 0"/>
-  <geometry>
-    <box size="0.1 0.01 0.12"/>
-  </geometry>
-</visual>
-<collision>
-  <origin rpy="1.57 -1.0 1.57" xyz="0 0 0"/>
-  <geometry>
-    <box size="0.1 0.01 0.12"/>
-  </geometry>
-</collision>
-<inertial>
-  <mass value="1"/>
-  <origin rpy="0 0 0" xyz="0 0 0"/>
-  <inertia ixx="1" ixy="0" ixz="0" iyy="1" iyz="0" izz="1"/>
-</inertial>
+  <visual>
+    <origin rpy="-1.0 1.57 1.57" xyz="0 0 0"/>
+    <geometry>
+      <box size="0.1 0.01 0.12"/>
+    </geometry>
+  </visual>
+  <collision>
+    <origin rpy="1.57 -1.0 1.57" xyz="0 0 0"/>
+    <geometry>
+      <box size="0.1 0.01 0.12"/>
+    </geometry>
+  </collision>
+  <inertial>
+    <mass value="1"/>
+    <origin rpy="0 0 0" xyz="0 0 0"/>
+    <inertia ixx="1" ixy="0" ixz="0" iyy="1" iyz="0" izz="1"/>
+  </inertial>
 </link>
 <link name="right_fence">
-<visual>
-  <origin rpy="1.57 1.0 1.57" xyz="0 0 0"/>
-  <geometry>
-    <box size="0.1 0.01 0.12"/>
-  </geometry>
-</visual>
-<collision>
-  <origin rpy="1.57 1.0 1.57" xyz="0 0 0"/>
-  <geometry>
-    <box size="0.1 0.01 0.12"/>
-  </geometry>
-</collision>
-<inertial>
-  <mass value="1"/>
-  <origin rpy="0 0 0" xyz="0 0 0"/>
-  <inertia ixx="1" ixy="0" ixz="0" iyy="1" iyz="0" izz="1"/>
-</inertial>
+  <visual>
+    <origin rpy="1.0 1.57 1.57" xyz="0 0 0"/>
+    <geometry>
+      <box size="0.1 0.01 0.12"/>
+    </geometry>
+  </visual>
+  <collision>
+    <origin rpy="1.57 1.0 1.57" xyz="0 0 0"/>
+    <geometry>
+      <box size="0.1 0.01 0.12"/>
+    </geometry>
+  </collision>
+  <inertial>
+    <mass value="1"/>
+    <origin rpy="0 0 0" xyz="0 0 0"/>
+    <inertia ixx="1" ixy="0" ixz="0" iyy="1" iyz="0" izz="1"/>
+  </inertial>
 </link>
 <link name="left_fence_front">
