Commit message: Converting controls to Twist messages, improving keyboard controls (robot can now both go forward or backward and left or right at the same time - circular motion)

File: malakrobo_description/urdf/malakrobo.xacro (robot description, xacro)
@@ -271,26 +271,26 @@
     </inertial>
   </link>
+  <link name="right_wheel">
+    <visual>
+      <origin rpy="1.57 0 0" xyz="0 0 0"/>
+      <geometry>
+        <cylinder radius="0.1" length="0.05"/>
+      </geometry>
+    </visual>
+    <collision>
+      <origin rpy="-1.57 0 0" xyz="0 0 0"/>
+      <geometry>
+        <cylinder radius="0.1" length="0.05"/>
+      </geometry>
+    </collision>
+    <inertial>
+      <mass value="5"/>
+      <origin rpy="0 0 0" xyz="0 0 0"/>
+      <inertia ixx="1" ixy="0" ixz="0" iyy="1" iyz="0" izz="1"/>
+    </inertial>
+  </link>
   <link name="left_wheel">
     <visual>
-      <origin rpy="1.57 0 0" xyz="0 0 0"/>
-      <geometry>
-        <cylinder radius="0.1" length="0.05"/>
-      </geometry>
-    </visual>
-    <collision>
-      <origin rpy="1.57 0 0" xyz="0 0 0"/>
-      <geometry>
-        <cylinder radius="0.1" length="0.05"/>
-      </geometry>
-    </collision>
-    <inertial>
-      <mass value="5"/>
-      <origin rpy="0 0 0" xyz="0 0 0"/>
-      <inertia ixx="1" ixy="0" ixz="0" iyy="1" iyz="0" izz="1"/>
-    </inertial>
-  </link>
-  <link name="right_wheel">
-    <visual>
-      <origin rpy="1.57 0 0" xyz="0 0 0"/>
+      <origin rpy="-1.57 0 0" xyz="0 0 0"/>
       <geometry>
         <cylinder radius="0.1" length="0.05"/>
@@ -371,5 +371,5 @@
   <joint name="sensor_base_joint" type="fixed">
     <axis xyz="0 0 0" />
-    <origin xyz="-0.15 0 0.20" rpy="0 0 0"/>
+    <origin xyz="0.15 0 0.20" rpy="0 0 3.14"/>
     <parent link="base_link"/>
     <child link="sensor_base"/>
@@ -377,5 +377,5 @@
   <joint name="camera_joint" type="fixed">
     <axis xyz="0 0 0" />
-    <origin xyz="-0.025 0 0.05" rpy="0 0 3.14"/>
+    <origin xyz="0.025 0 0.05" rpy="0 0 3.14"/>
     <parent link="sensor_base"/>
     <child link="camera"/>
@@ -394,5 +394,5 @@
   </joint>
   <joint name="base2_joint" type="fixed">
-    <origin rpy="0 0 0" xyz="-0.15 0 0"/>
+    <origin rpy="0 0 0" xyz="0.15 0 0"/>
     <parent link="base_link"/>
     <child link="base3"/>
@@ -400,5 +400,5 @@
   </joint>
   <joint name="base3_base_fence_joint" type="fixed">
-    <origin rpy="0 0 0" xyz="-0.075 0 0"/>
+    <origin rpy="0 0 0" xyz="0.075 0 0"/>
     <parent link="base3"/>
     <child link="base_fence"/>
@@ -406,5 +406,5 @@
   </joint>
   <joint name="base_to_left_fence" type="fixed">
-    <origin rpy="0 0 0" xyz="-0.055 -0.15 0.1"/>
+    <origin rpy="0 0 0" xyz="0.055 0.15 0.1"/>
     <parent link="base_fence"/>
     <child link="left_fence"/>
@@ -412,5 +412,5 @@
   </joint>
   <joint name="base_to_right_fence" type="fixed">
-    <origin rpy="0 0 0" xyz="-0.055 0.15 0.1"/>
+    <origin rpy="0 0 0" xyz="0.055 -0.15 0.1"/>
     <parent link="base_fence"/>
     <child link="right_fence"/>
@@ -418,5 +418,5 @@
   </joint>
   <joint name="left_fence_to_front" type="fixed">
-    <origin rpy="0 0 0" xyz="-0.0855 -0.035 0.0"/>
+    <origin rpy="0 0 0" xyz="0.0855 0.035 0.0"/>
     <parent link="left_fence"/>
     <child link="left_fence_front"/>
@@ -424,5 +424,5 @@
   </joint>
   <joint name="right_fence_to_front" type="fixed">
-    <origin rpy="0 0 0" xyz="-0.0855 0.035 0.0"/>
+    <origin rpy="0 0 0" xyz="0.0855 -0.035 0.0"/>
     <parent link="right_fence"/>
     <child link="right_fence_front"/>
@@ -465,17 +465,27 @@
     <axis xyz="0.0 1.0 0.0"/>
   </joint>
-  <joint name="base_to_left_wheel" type="continuous">
+  <joint name="base_to_right_wheel" type="continuous">
     <origin rpy="0 0 0" xyz="0 -0.225 0.1"/>
     <parent link="base2"/>
-    <child link="left_wheel"/>
-    <axis xyz="0.0 1.0 0.0"/>
-  </joint>
-  <joint name="base_to_right_wheel" type="continuous">
+    <child link="right_wheel"/>
+    <axis xyz="0.0 1.0 0.0"/>
+  </joint>
+  <joint name="base_to_left_wheel" type="continuous">
     <origin rpy="0 0 0" xyz="0 0.225 0.1"/>
     <parent link="base2"/>
-    <child link="right_wheel"/>
+    <child link="left_wheel"/>
     <axis xyz="0.0 1.0 0.0"/>
   </joint>
   <transmission name="tran1">
+    <type>transmission_interface/SimpleTransmission</type>
+    <joint name="base_to_right_wheel">
+      <hardwareInterface>EffortJointInterface</hardwareInterface>
+    </joint>
+    <actuator name="right_wheel">
+      <hardwareInterface>EffortJointInterface</hardwareInterface>
+      <mechanicalReduction>1</mechanicalReduction>
+    </actuator>
+  </transmission>
+  <transmission name="tran2">
     <type>transmission_interface/SimpleTransmission</type>
     <joint name="base_to_left_wheel">
@@ -487,13 +497,3 @@
     </actuator>
   </transmission>
-  <transmission name="tran2">
-    <type>transmission_interface/SimpleTransmission</type>
-    <joint name="base_to_right_wheel">
-      <hardwareInterface>EffortJointInterface</hardwareInterface>
-    </joint>
-    <actuator name="right_wheel">
-      <hardwareInterface>EffortJointInterface</hardwareInterface>
-      <mechanicalReduction>1</mechanicalReduction>
-    </actuator>
-  </transmission>
 </robot>

Commit message: Fixing control and mapping

File: malakrobo_description/urdf/malakrobo.xacro (robot description, xacro)
@@ -5,24 +5,24 @@
   <xacro:include filename="$(find malakrobo_description)/urdf/materials.xacro" />
   <xacro:include filename="$(find malakrobo_description)/urdf/malakrobo.gazebo" />
+  <link name="base2">
+    <visual>
+      <origin rpy="0 0 0" xyz="0 0 0.1"/>
+      <geometry>
+        <cylinder radius="0.2" length="0.02"/>
+      </geometry>
+    </visual>
+    <collision>
+      <origin rpy="0 0 0" xyz="0 0 0.1"/>
+      <geometry>
+        <cylinder radius="0.2" length="0.02"/>
+      </geometry>
+    </collision>
+    <inertial>
+      <mass value="5"/>
+      <origin rpy="0 0 0" xyz="0 0 0"/>
+      <inertia ixx="1" ixy="0" ixz="0" iyy="1" iyz="0" izz="1"/>
+    </inertial>
+  </link>
   <link name="base_link">
-    <visual>
-      <origin rpy="0 0 0" xyz="0 0 0.1"/>
-      <geometry>
-        <cylinder radius="0.2" length="0.02"/>
-      </geometry>
-    </visual>
-    <collision>
-      <origin rpy="0 0 0" xyz="0 0 0.1"/>
-      <geometry>
-        <cylinder radius="0.2" length="0.02"/>
-      </geometry>
-    </collision>
-    <inertial>
-      <mass value="5"/>
-      <origin rpy="0 0 0" xyz="0 0 0"/>
-      <inertia ixx="1" ixy="0" ixz="0" iyy="1" iyz="0" izz="1"/>
-    </inertial>
-  </link>
-  <link name="base2">
     <visual>
       <origin rpy="0 0 0" xyz="0 0 0.1"/>
@@ -372,5 +372,5 @@
     <axis xyz="0 0 0" />
     <origin xyz="0.15 0 0.20" rpy="0 0 3.14"/>
-    <parent link="base_link"/>
+    <parent link="base2"/>
     <child link="sensor_base"/>
   </joint>
@@ -395,5 +395,5 @@
   <joint name="base2_joint" type="fixed">
     <origin rpy="0 0 0" xyz="0.15 0 0"/>
-    <parent link="base_link"/>
+    <parent link="base2"/>
     <child link="base3"/>
     <axis xyz="0.0 0.0 0.0"/>
@@ -431,5 +431,5 @@
   <joint name="front_caster_base_joint" type="continuous">
     <origin rpy="0 0 0" xyz="0.15 0 0.08"/>
-    <parent link="base_link"/>
+    <parent link="base2"/>
     <child link="front_caster_base"/>
     <axis xyz="0.0 0.0 1.0"/>
@@ -437,5 +437,5 @@
   <joint name="back_caster_base_joint" type="continuous">
     <origin rpy="0 0 0" xyz="-0.15 0 0.08"/>
-    <parent link="base_link"/>
+    <parent link="base2"/>
     <child link="back_caster_base"/>
     <axis xyz="0.0 0.0 1.0"/>
@@ -467,5 +467,5 @@
   <joint name="base_to_right_wheel" type="continuous">
     <origin rpy="0 0 0" xyz="0 -0.225 0.1"/>
-    <parent link="base2"/>
+    <parent link="base_link"/>
     <child link="right_wheel"/>
     <axis xyz="0.0 1.0 0.0"/>
@@ -473,5 +473,5 @@
   <joint name="base_to_left_wheel" type="continuous">
     <origin rpy="0 0 0" xyz="0 0.225 0.1"/>
-    <parent link="base2"/>
+    <parent link="base_link"/>
     <child link="left_wheel"/>
     <axis xyz="0.0 1.0 0.0"/>
@@ -480,20 +480,70 @@
     <type>transmission_interface/SimpleTransmission</type>
     <joint name="base_to_right_wheel">
-      <hardwareInterface>EffortJointInterface</hardwareInterface>
+      <hardwareInterface>hardware_interface/VelocityJointInterface</hardwareInterface>
     </joint>
     <actuator name="right_wheel">
+      <hardwareInterface>VelocityJointInterface</hardwareInterface>
+      <mechanicalReduction>7</mechanicalReduction>
+    </actuator>
+  </transmission>
+  <transmission name="tran2">
+    <type>transmission_interface/SimpleTransmission</type>
+    <joint name="base_to_left_wheel">
+      <hardwareInterface>hardware_interface/VelocityJointInterface</hardwareInterface>
+    </joint>
+    <actuator name="left_wheel">
+      <hardwareInterface>VelocityJointInterface</hardwareInterface>
+      <mechanicalReduction>7</mechanicalReduction>
+    </actuator>
+  </transmission>
+  <transmission name="tran3">
+    <type>transmission_interface/SimpleTransmission</type>
+    <joint name="front_caster_base_joint">
+      <hardwareInterface>EffortJointInterface</hardwareInterface>
+    </joint>
+    <actuator name="front_caster_base">
       <hardwareInterface>EffortJointInterface</hardwareInterface>
       <mechanicalReduction>1</mechanicalReduction>
     </actuator>
   </transmission>
-  <transmission name="tran2">
-    <type>transmission_interface/SimpleTransmission</type>
-    <joint name="base_to_left_wheel">
-      <hardwareInterface>EffortJointInterface</hardwareInterface>
-    </joint>
-    <actuator name="left_wheel">
+  <transmission name="tran3">
+    <type>transmission_interface/SimpleTransmission</type>
+    <joint name="front_caster_base_joint">
+      <hardwareInterface>EffortJointInterface</hardwareInterface>
+    </joint>
+    <actuator name="front_caster_base">
       <hardwareInterface>EffortJointInterface</hardwareInterface>
       <mechanicalReduction>1</mechanicalReduction>
     </actuator>
   </transmission>
+  <transmission name="tran4">
+    <type>transmission_interface/SimpleTransmission</type>
+    <joint name="back_caster_base_joint">
+      <hardwareInterface>EffortJointInterface</hardwareInterface>
+    </joint>
+    <actuator name="back_caster_base">
+      <hardwareInterface>EffortJointInterface</hardwareInterface>
+      <mechanicalReduction>1</mechanicalReduction>
+    </actuator>
+  </transmission>
+    <transmission name="tran5">
+    <type>transmission_interface/SimpleTransmission</type>
+    <joint name="front_caster_wheel_joint">
+      <hardwareInterface>EffortJointInterface</hardwareInterface>
+    </joint>
+    <actuator name="front_caster_wheel">
+      <hardwareInterface>EffortJointInterface</hardwareInterface>
+      <mechanicalReduction>1</mechanicalReduction>
+    </actuator>
+  </transmission>
+  <transmission name="tran6">
+    <type>transmission_interface/SimpleTransmission</type>
+    <joint name="back_caster_wheel_joint">
+      <hardwareInterface>EffortJointInterface</hardwareInterface>
+    </joint>
+    <actuator name="back_caster_wheel">
+      <hardwareInterface>EffortJointInterface</hardwareInterface>
+      <mechanicalReduction>1</mechanicalReduction>
+    </actuator>
+  </transmission>
 </robot>

Commit message: Fixing diff drive, removing drift fixing the wheel separation which resulted in wrong angles

File: malakrobo_description/urdf/malakrobo.xacro (robot description, xacro)
@@ -19,5 +19,5 @@
     </collision>
     <inertial>
-      <mass value="5"/>
+      <mass value="100"/>
       <origin rpy="0 0 0" xyz="0 0 0"/>
       <inertia ixx="1" ixy="0" ixz="0" iyy="1" iyz="0" izz="1"/>
@@ -38,5 +38,5 @@
     </collision>
     <inertial>
-      <mass value="5"/>
+      <mass value="100"/>
       <origin rpy="0 0 0" xyz="0 0 0"/>
       <inertia ixx="1" ixy="0" ixz="0" iyy="1" iyz="0" izz="1"/>
@@ -285,7 +285,7 @@
     </collision>
     <inertial>
-      <mass value="5"/>
-      <origin rpy="0 0 0" xyz="0 0 0"/>
-      <inertia ixx="1" ixy="0" ixz="0" iyy="1" iyz="0" izz="1"/>
+      <mass value="10"/>
+      <origin rpy="0 0 0" xyz="0 0 0"/>
+      <inertia ixx="0.027" ixy="0" ixz="0" iyy="0.027" iyz="0" izz="0.05"/>
     </inertial>
   </link>
@@ -304,7 +304,7 @@
     </collision>
     <inertial>
-      <mass value="5"/>
-      <origin rpy="0 0 0" xyz="0 0 0"/>
-      <inertia ixx="1" ixy="0" ixz="0" iyy="1" iyz="0" izz="1"/>
+      <mass value="10"/>
+      <origin rpy="0 0 0" xyz="0 0 0"/>
+      <inertia ixx="0.027" ixy="0" ixz="0" iyy="0.027" iyz="0" izz="0.05"/>
     </inertial>
   </link>

Commit message: Tweaks to navigation stack, adding automated movement between preselected points (read from file, can be executed one by one after user action or one by one when the previous target is reached

File: malakrobo_description/urdf/malakrobo.xacro (robot description, xacro)
@@ -371,5 +371,5 @@
   <joint name="sensor_base_joint" type="fixed">
     <axis xyz="0 0 0" />
-    <origin xyz="0.15 0 0.20" rpy="0 0 3.14"/>
+    <origin xyz="0 0 0.20" rpy="0 0 3.14"/>
     <parent link="base2"/>
     <child link="sensor_base"/>
@@ -377,5 +377,5 @@
   <joint name="camera_joint" type="fixed">
     <axis xyz="0 0 0" />
-    <origin xyz="0.025 0 0.05" rpy="0 0 3.14"/>
+    <origin xyz="-0.025 0 0.05" rpy="0 0 3.14"/>
     <parent link="sensor_base"/>
     <child link="camera"/>

Commit message: Finalizing navigation stack, upgrading to LIDAR (previously hokuyo sensor). Adjusting camera for better image quality, starting testing find_object_2d to recognize balls

File: malakrobo_description/urdf/malakrobo.xacro (robot description, xacro)
@@ -313,5 +313,5 @@
       <origin xyz="0 0 0" rpy="0 0 0"/>
       <geometry>
-        <box size="0.1 0.1 0.2"/>
+        <box size="0.1 0.1 0.23"/>
       </geometry>
     </collision>
@@ -319,5 +319,5 @@
       <origin xyz="0 0 0" rpy="0 0 0"/>
       <geometry>
-        <box size="0.05 0.05 0.2"/>
+        <box size="0.05 0.05 0.21"/>
       </geometry>
     </visual>
@@ -349,27 +349,26 @@
     </inertial>
   </link>
-  <!-- Hokuyo Laser -->
-  <link name="hokuyo">
-    <collision>
-      <origin xyz="0 0 0" rpy="0 0 0"/>
-      <geometry>
-        <box size="0.1 0.1 0.1"/>
-      </geometry>
-    </collision>
-    <visual>
-      <origin xyz="0 0 0" rpy="0 0 0"/>
-      <geometry>
-        <mesh filename="package://malakrobo_description/meshes/hokuyo.dae"/>
+  <link name="laser">
+    <collision>
+      <origin xyz="0 0 0" rpy="1.5707 0 4.71"/>
+      <geometry>
+        <mesh filename="package://malakrobo_description/meshes/rplidar.dae" scale="0.001 0.001 0.001" />
+      </geometry>
+    </collision>
+    <visual>
+      <origin xyz="0 0 0" rpy="1.5707 0 4.71"/>
+      <geometry>
+        <mesh filename="package://malakrobo_description/meshes/rplidar.dae" scale="0.001 0.001 0.001" />
       </geometry>
     </visual>
     <inertial>
       <mass value="1e-5" />
-      <origin xyz="0 0 0" rpy="0 0 0"/>
-      <inertia ixx="1e-6" ixy="0" ixz="0" iyy="1e-6" iyz="0" izz="1e-6" />
+      <origin xyz="0 0 0" rpy="1.5707 0 4.71"/>
+      <inertia ixx="0" ixy="0" ixz="0" iyy="0" iyz="0" izz="0" />
     </inertial>
   </link>
   <joint name="sensor_base_joint" type="fixed">
     <axis xyz="0 0 0" />
-    <origin xyz="0 0 0.20" rpy="0 0 3.14"/>
+    <origin xyz="0 0 0.23" rpy="0 0 3.14"/>
     <parent link="base2"/>
     <child link="sensor_base"/>
@@ -381,9 +380,9 @@
     <child link="camera"/>
   </joint>
-  <joint name="hokuyo_joint" type="fixed">
+  <joint name="rplidar_joint" type="fixed">
     <axis xyz="0 1 0" />
-    <origin xyz="0 0 0.13" rpy="0 0 3.14"/>
+    <origin xyz="0 0 0.10" rpy="0 0 3.14"/>
     <parent link="sensor_base"/>
-    <child link="hokuyo"/>
+    <child link="laser"/>
   </joint>
   <joint name="base_joint" type="fixed">

Commit message: Movable arms, controller for arms, attempt to automatically close grippers

File: malakrobo_description/urdf/malakrobo.xacro (robot description, xacro)
@@ -121,13 +121,13 @@
   <link name="left_fence_front">
   <visual>
-  <origin rpy="1.5 1.57 1.57" xyz="0 0 0"/>
+  <origin rpy="1.57 1.57 1.57" xyz="0.1 0 0"/>
   <geometry>
-    <box size="0.1 0.01 0.075"/>
+    <box size="0.1 0.01 0.2"/>
   </geometry>
   </visual>
   <collision>
-  <origin rpy="1.57 -1.5 1.57" xyz="0 0 0"/>
+  <origin rpy="1.57 -1.5 1.57" xyz="0.1 0 0"/>
   <geometry>
-    <box size="0.1 0.01 0.075"/>
+    <box size="0.1 0.01 0.2"/>
   </geometry>
   </collision>
@@ -140,13 +140,13 @@
   <link name="right_fence_front">
   <visual>
-  <origin rpy="-1.5 1.57 1.57" xyz="0 0 0"/>
+  <origin rpy="-1.57 1.57 1.57" xyz="0.1 0 0"/>
   <geometry>
-    <box size="0.1 0.01 0.075"/>
+    <box size="0.1 0.01 0.2"/>
   </geometry>
   </visual>
   <collision>
-  <origin rpy="1.57 1.5 1.57" xyz="0 0 0"/>
+  <origin rpy="1.57 1.5 1.57" xyz="0.1 0 0"/>
   <geometry>
-    <box size="0.1 0.01 0.075"/>
+    <box size="0.1 0.01 0.2"/>
   </geometry>
   </collision>
@@ -416,15 +416,15 @@
     <axis xyz="0.0 1.0 0.0"/>
   </joint>
-  <joint name="left_fence_to_front" type="fixed">
-    <origin rpy="0 0 0" xyz="0.0855 0.035 0.0"/>
+  <joint name="left_fence_to_front" type="continuous">
+    <origin rpy="0 0 0" xyz="0.045 0.030 0.0"/>
     <parent link="left_fence"/>
     <child link="left_fence_front"/>
-    <axis xyz="0.0 1.0 0.0"/>
-  </joint>
-  <joint name="right_fence_to_front" type="fixed">
-    <origin rpy="0 0 0" xyz="0.0855 -0.035 0.0"/>
+    <axis xyz="0.0 0.0 1.0"/>
+  </joint>
+  <joint name="right_fence_to_front" type="continuous">
+    <origin rpy="0 0 0" xyz="0.045 -0.030 0.0"/>
     <parent link="right_fence"/>
     <child link="right_fence_front"/>
-    <axis xyz="0.0 1.0 0.0"/>
+    <axis xyz="0.0 0.0 1.0"/>
   </joint>
   <joint name="front_caster_base_joint" type="continuous">
@@ -546,3 +546,21 @@
     </actuator>
   </transmission>
+  <transmission name="tran7">
+    <type>transmission_interface/SimpleTransmission</type>
+    <joint name="left_fence_to_front">
+      <hardwareInterface>EffortJointInterface</hardwareInterface>
+    </joint>
+    <actuator name="left_fence_front">
+      <hardwareInterface>EffortJointInterface</hardwareInterface>
+    </actuator>
+  </transmission>
+  <transmission name="tran8">
+    <type>transmission_interface/SimpleTransmission</type>
+    <joint name="right_fence_to_front">
+      <hardwareInterface>EffortJointInterface</hardwareInterface>
+    </joint>
+    <actuator name="right_fence_front">
+      <hardwareInterface>EffortJointInterface</hardwareInterface>
+    </actuator>
+  </transmission>
 </robot>

Commit message: Disabling grippers as they cause errors, currently in fixed state

File: malakrobo_description/urdf/malakrobo.xacro (robot description, xacro)
@@ -416,5 +416,5 @@
     <axis xyz="0.0 1.0 0.0"/>
   </joint>
-  <joint name="left_fence_to_front" type="continuous">
+  <joint name="left_fence_to_front" type="fixed">
     <origin rpy="0 0 0" xyz="0.045 0.030 0.0"/>
     <parent link="left_fence"/>
@@ -422,5 +422,5 @@
     <axis xyz="0.0 0.0 1.0"/>
   </joint>
-  <joint name="right_fence_to_front" type="continuous">
+  <joint name="right_fence_to_front" type="fixed">
     <origin rpy="0 0 0" xyz="0.045 -0.030 0.0"/>
     <parent link="right_fence"/>
@@ -546,21 +546,21 @@
     </actuator>
   </transmission>
-  <transmission name="tran7">
-    <type>transmission_interface/SimpleTransmission</type>
-    <joint name="left_fence_to_front">
-      <hardwareInterface>EffortJointInterface</hardwareInterface>
-    </joint>
-    <actuator name="left_fence_front">
-      <hardwareInterface>EffortJointInterface</hardwareInterface>
-    </actuator>
-  </transmission>
-  <transmission name="tran8">
-    <type>transmission_interface/SimpleTransmission</type>
-    <joint name="right_fence_to_front">
-      <hardwareInterface>EffortJointInterface</hardwareInterface>
-    </joint>
-    <actuator name="right_fence_front">
-      <hardwareInterface>EffortJointInterface</hardwareInterface>
-    </actuator>
-  </transmission>
+<!--  <transmission name="tran7">-->
+<!--    <type>transmission_interface/SimpleTransmission</type>-->
+<!--    <joint name="left_fence_to_front">-->
+<!--      <hardwareInterface>EffortJointInterface</hardwareInterface>-->
+<!--    </joint>-->
+<!--    <actuator name="left_fence_front">-->
+<!--      <hardwareInterface>EffortJointInterface</hardwareInterface>-->
+<!--    </actuator>-->
+<!--  </transmission>-->
+<!--  <transmission name="tran8">-->
+<!--    <type>transmission_interface/SimpleTransmission</type>-->
+<!--    <joint name="right_fence_to_front">-->
+<!--      <hardwareInterface>EffortJointInterface</hardwareInterface>-->
+<!--    </joint>-->
+<!--    <actuator name="right_fence_front">-->
+<!--      <hardwareInterface>EffortJointInterface</hardwareInterface>-->
+<!--    </actuator>-->
+<!--  </transmission>-->
 </robot>

Commit message: Adding GUI, implementing different autonomy stages, working on correct TFs

File: malakrobo_description/urdf/malakrobo.xacro (robot description, xacro)
@@ -330,5 +330,5 @@
   <link name="camera">
     <collision>
-      <origin xyz="0 0 0" rpy="0 0 0"/>
+      <origin xyz="0 0 0" rpy="0 0 0.0"/>
       <geometry>
         <box size="${cameraSize} ${cameraSize} ${cameraSize}"/>
@@ -336,5 +336,5 @@
     </collision>
     <visual>
-      <origin xyz="0 0 0" rpy="0 0 0"/>
+      <origin xyz="0 0 0" rpy="0 0 0.0"/>
       <geometry>
         <box size="${cameraSize} ${cameraSize} ${cameraSize}"/>
@@ -344,5 +344,5 @@
     <inertial>
       <mass value="${cameraMass}" />
-      <origin xyz="0 0 0" rpy="0 0 0"/>
+      <origin xyz="0 0 0" rpy="0 0 0.0"/>
       <box_inertia m="${cameraMass}" x="${cameraSize}" y="${cameraSize}" z="${cameraSize}" />
       <inertia ixx="1e-6" ixy="0" ixz="0" iyy="1e-6" iyz="0" izz="1e-6" />
