Commit message: Implementing most of the autonomous features, adding vacuum effector (for grabbing balls), implementing go home and drop the ball, implementing object recognition with automatic ball grabbing, optimising paths, modifying the visuals of the robot, TODO: Go to each objects and grab it, full path, tiny fixes to path optimisation

File: malakrobo_description/urdf/malakrobo.xacro (robot description, xacro)
@@ -1,566 +1,603 @@
 <?xml version="1.0" ?>
 <robot name="malakrobo" xmlns:xacro="http://www.ros.org/wiki/xacro">
-  <xacro:property name="cameraSize" value="0.05"/>
-  <xacro:property name="cameraMass" value="0.1"/>
-  <xacro:include filename="$(find malakrobo_description)/urdf/materials.xacro" />
-  <xacro:include filename="$(find malakrobo_description)/urdf/malakrobo.gazebo" />
-  <link name="base2">
-    <visual>
-      <origin rpy="0 0 0" xyz="0 0 0.1"/>
-      <geometry>
-        <cylinder radius="0.2" length="0.02"/>
-      </geometry>
-    </visual>
-    <collision>
-      <origin rpy="0 0 0" xyz="0 0 0.1"/>
-      <geometry>
-        <cylinder radius="0.2" length="0.02"/>
-      </geometry>
-    </collision>
-    <inertial>
-      <mass value="100"/>
-      <origin rpy="0 0 0" xyz="0 0 0"/>
-      <inertia ixx="1" ixy="0" ixz="0" iyy="1" iyz="0" izz="1"/>
-    </inertial>
-  </link>
-  <link name="base_link">
-    <visual>
-      <origin rpy="0 0 0" xyz="0 0 0.1"/>
-      <geometry>
-        <box size="0.1 0.4 0.02"/>
-      </geometry>
-    </visual>
-    <collision>
-      <origin rpy="0 0 0" xyz="0 0 0.1"/>
-      <geometry>
-        <box size="0.1 0.4 0.02"/>
-      </geometry>
-    </collision>
-    <inertial>
-      <mass value="100"/>
-      <origin rpy="0 0 0" xyz="0 0 0"/>
-      <inertia ixx="1" ixy="0" ixz="0" iyy="1" iyz="0" izz="1"/>
-    </inertial>
-  </link>
-  <link name="base3">
-    <visual>
-      <origin rpy="0 0 0" xyz="0 0 0.1"/>
-      <geometry>
-        <box size="0.15 0.25 0.02"/>
-      </geometry>
-    </visual>
-    <collision>
-      <origin rpy="0 0 0" xyz="0 0 0.1"/>
-      <geometry>
-        <box size="0.15 0.25 0.02"/>
-      </geometry>
-    </collision>
-    <inertial>
-      <mass value="1"/>
-      <origin rpy="0 0 0" xyz="0 0 0"/>
-      <inertia ixx="1" ixy="0" ixz="0" iyy="1" iyz="0" izz="1"/>
-    </inertial>
-  </link>
-  <link name="base_fence">
-    <visual>
-      <origin rpy="0 0 0" xyz="0 0 0.1"/>
-      <geometry>
-        <box size="0.02 0.25 0.1"/>
-      </geometry>
-    </visual>
-    <collision>
-      <origin rpy="0 0 0" xyz="0 0 0.1"/>
-      <geometry>
-        <box size="0.02 0.25 0.1"/>
-      </geometry>
-    </collision>
-    <inertial>
-      <mass value="1"/>
-      <origin rpy="0 0 0" xyz="0 0 0"/>
-      <inertia ixx="1" ixy="0" ixz="0" iyy="1" iyz="0" izz="1"/>
-    </inertial>
-  </link>
-  <link name="left_fence">
-    <visual>
-      <origin rpy="1.0 1.57 1.57" xyz="0 0 0"/>
-      <geometry>
-        <box size="0.1 0.01 0.12"/>
-      </geometry>
-    </visual>
-    <collision>
-      <origin rpy="1.57 -1.0 1.57" xyz="0 0 0"/>
-      <geometry>
-        <box size="0.1 0.01 0.12"/>
-      </geometry>
-    </collision>
-    <inertial>
-      <mass value="1"/>
-      <origin rpy="0 0 0" xyz="0 0 0"/>
-      <inertia ixx="1" ixy="0" ixz="0" iyy="1" iyz="0" izz="1"/>
-    </inertial>
-  </link>
-  <link name="right_fence">
-    <visual>
-      <origin rpy="-1.0 1.57 1.57" xyz="0 0 0"/>
-      <geometry>
-        <box size="0.1 0.01 0.12"/>
-      </geometry>
-    </visual>
-    <collision>
-      <origin rpy="1.57 1.0 1.57" xyz="0 0 0"/>
-      <geometry>
-        <box size="0.1 0.01 0.12"/>
-      </geometry>
-    </collision>
-    <inertial>
-      <mass value="1"/>
-      <origin rpy="0 0 0" xyz="0 0 0"/>
-      <inertia ixx="1" ixy="0" ixz="0" iyy="1" iyz="0" izz="1"/>
-    </inertial>
-  </link>
-  <link name="left_fence_front">
-  <visual>
-  <origin rpy="1.57 1.57 1.57" xyz="0.1 0 0"/>
-  <geometry>
-    <box size="0.1 0.01 0.2"/>
-  </geometry>
-  </visual>
-  <collision>
-  <origin rpy="1.57 -1.5 1.57" xyz="0.1 0 0"/>
-  <geometry>
-    <box size="0.1 0.01 0.2"/>
-  </geometry>
-  </collision>
-  <inertial>
-    <mass value="1"/>
-    <origin rpy="0 0 0" xyz="0 0 0"/>
-    <inertia ixx="1" ixy="0" ixz="0" iyy="1" iyz="0" izz="1"/>
-  </inertial>
-  </link>
-  <link name="right_fence_front">
-  <visual>
-  <origin rpy="-1.57 1.57 1.57" xyz="0.1 0 0"/>
-  <geometry>
-    <box size="0.1 0.01 0.2"/>
-  </geometry>
-  </visual>
-  <collision>
-  <origin rpy="1.57 1.5 1.57" xyz="0.1 0 0"/>
-  <geometry>
-    <box size="0.1 0.01 0.2"/>
-  </geometry>
-  </collision>
-  <inertial>
-    <mass value="1"/>
-    <origin rpy="0 0 0" xyz="0 0 0"/>
-    <inertia ixx="1" ixy="0" ixz="0" iyy="1" iyz="0" izz="1"/>
-  </inertial>
-  </link>
-  <link name="front_caster_base">
-    <visual>
-      <origin rpy="0 0 0" xyz="0 0 0"/>
-      <geometry>
-        <box size="0.075 0.075 0.02"/>
-      </geometry>
-    </visual>
-    <collision>
-      <origin rpy="0 0 0" xyz="0 0 0"/>
-      <geometry>
-        <box size="0.075 0.075 0.02"/>
-      </geometry>
-    </collision>
-    <inertial>
-      <mass value="0.5"/>
-      <origin rpy="0 0 0" xyz="0 0 0"/>
-      <inertia ixx="1" ixy="0" ixz="0" iyy="1" iyz="0" izz="1"/>
-    </inertial>
-  </link>
-  <link name="back_caster_base">
-    <visual>
-      <origin rpy="0 0 0" xyz="0 0 0"/>
-      <geometry>
-        <box size="0.075 0.075 0.02"/>
-      </geometry>
-    </visual>
-    <collision>
-      <origin rpy="0 0 0" xyz="0 0 0"/>
-      <geometry>
-        <box size="0.075 0.075 0.02"/>
-      </geometry>
-    </collision>
-    <inertial>
-      <mass value="0.5"/>
-      <origin rpy="0 0 0" xyz="0 0 0"/>
-      <inertia ixx="1" ixy="0" ixz="0" iyy="1" iyz="0" izz="1"/>
-    </inertial>
-  </link>
-  <link name="front_caster_side">
-    <visual>
-      <origin rpy="0 0 0" xyz="0 0 0"/>
-      <geometry>
-        <box size="0.075 0.02 0.05"/>
-      </geometry>
-    </visual>
-    <collision>
-      <origin rpy="0 0 0" xyz="0 0 0"/>
-      <geometry>
-        <box size="0.075 0.02 0.05"/>
-      </geometry>
-    </collision>
-    <inertial>
-      <mass value="0.5"/>
-      <origin rpy="0 0 0" xyz="0 0 0"/>
-      <inertia ixx="1" ixy="0" ixz="0" iyy="1" iyz="0" izz="1"/>
-    </inertial>
-  </link>
-  <link name="back_caster_side">
-    <visual>
-      <origin rpy="0 0 0" xyz="0 0 0"/>
-      <geometry>
-        <box size="0.075 0.02 0.05"/>
-      </geometry>
-    </visual>
-    <collision>
-      <origin rpy="0 0 0" xyz="0 0 0"/>
-      <geometry>
-        <box size="0.075 0.02 0.05"/>
-      </geometry>
-    </collision>
-    <inertial>
-      <mass value="0.5"/>
-      <origin rpy="0 0 0" xyz="0 0 0"/>
-      <inertia ixx="1" ixy="0" ixz="0" iyy="1" iyz="0" izz="1"/>
-    </inertial>
-  </link>
-  <link name="front_caster_wheel">
-    <visual>
-      <origin rpy="1.57 0 0" xyz="0 0 0"/>
-      <geometry>
-        <cylinder radius="0.03" length="0.035"/>
-      </geometry>
-    </visual>
-    <collision>
-      <origin rpy="1.57 0 0" xyz="0 0 0"/>
-      <geometry>
-        <cylinder radius="0.03" length="0.035"/>
-      </geometry>
-    </collision>
-    <inertial>
-      <mass value="5"/>
-      <origin rpy="0 0 0" xyz="0 0 0"/>
-      <inertia ixx="1" ixy="0" ixz="0" iyy="1" iyz="0" izz="1"/>
-    </inertial>
-  </link>
-  <link name="back_caster_wheel">
-    <visual>
-      <origin rpy="-1.57 0 0" xyz="0 0 0"/>
-      <geometry>
-        <cylinder radius="0.03" length="0.035"/>
-      </geometry>
-    </visual>
-    <collision>
-      <origin rpy="-1.57 0 0" xyz="0 0 0"/>
-      <geometry>
-        <cylinder radius="0.03" length="0.035"/>
-      </geometry>
-    </collision>
-    <inertial>
-      <mass value="5"/>
-      <origin rpy="0 0 0" xyz="0 0 0"/>
-      <inertia ixx="1" ixy="0" ixz="0" iyy="1" iyz="0" izz="1"/>
-    </inertial>
-  </link>
-  <link name="right_wheel">
-    <visual>
-      <origin rpy="1.57 0 0" xyz="0 0 0"/>
-      <geometry>
-        <cylinder radius="0.1" length="0.05"/>
-      </geometry>
-    </visual>
-    <collision>
-      <origin rpy="-1.57 0 0" xyz="0 0 0"/>
-      <geometry>
-        <cylinder radius="0.1" length="0.05"/>
-      </geometry>
-    </collision>
-    <inertial>
-      <mass value="10"/>
-      <origin rpy="0 0 0" xyz="0 0 0"/>
-      <inertia ixx="0.027" ixy="0" ixz="0" iyy="0.027" iyz="0" izz="0.05"/>
-    </inertial>
-  </link>
-  <link name="left_wheel">
-    <visual>
-      <origin rpy="-1.57 0 0" xyz="0 0 0"/>
-      <geometry>
-        <cylinder radius="0.1" length="0.05"/>
-      </geometry>
-    </visual>
-    <collision>
-      <origin rpy="1.57 0 0" xyz="0 0 0"/>
-      <geometry>
-        <cylinder radius="0.1" length="0.05"/>
-      </geometry>
-    </collision>
-    <inertial>
-      <mass value="10"/>
-      <origin rpy="0 0 0" xyz="0 0 0"/>
-      <inertia ixx="0.027" ixy="0" ixz="0" iyy="0.027" iyz="0" izz="0.05"/>
-    </inertial>
-  </link>
-  <link name="sensor_base">
-    <collision>
-      <origin xyz="0 0 0" rpy="0 0 0"/>
-      <geometry>
-        <box size="0.1 0.1 0.23"/>
-      </geometry>
-    </collision>
-    <visual>
-      <origin xyz="0 0 0" rpy="0 0 0"/>
-      <geometry>
-        <box size="0.05 0.05 0.21"/>
-      </geometry>
-    </visual>
-    <inertial>
-      <mass value="1e-5" />
-      <origin xyz="0 0 0" rpy="0 0 0"/>
-      <inertia ixx="1e-6" ixy="0" ixz="0" iyy="1e-6" iyz="0" izz="1e-6" />
-    </inertial>
-  </link>
-  <link name="camera">
-    <collision>
-      <origin xyz="0 0 0" rpy="0 0 0.0"/>
-      <geometry>
-        <box size="${cameraSize} ${cameraSize} ${cameraSize}"/>
-      </geometry>
-    </collision>
-    <visual>
-      <origin xyz="0 0 0" rpy="0 0 0.0"/>
-      <geometry>
-        <box size="${cameraSize} ${cameraSize} ${cameraSize}"/>
-      </geometry>
-      <material name="green"/>
-    </visual>
-    <inertial>
-      <mass value="${cameraMass}" />
-      <origin xyz="0 0 0" rpy="0 0 0.0"/>
-      <box_inertia m="${cameraMass}" x="${cameraSize}" y="${cameraSize}" z="${cameraSize}" />
-      <inertia ixx="1e-6" ixy="0" ixz="0" iyy="1e-6" iyz="0" izz="1e-6" />
-    </inertial>
-  </link>
-  <link name="laser">
-    <collision>
-      <origin xyz="0 0 0" rpy="1.5707 0 4.71"/>
-      <geometry>
-        <mesh filename="package://malakrobo_description/meshes/rplidar.dae" scale="0.001 0.001 0.001" />
-      </geometry>
-    </collision>
-    <visual>
-      <origin xyz="0 0 0" rpy="1.5707 0 4.71"/>
-      <geometry>
-        <mesh filename="package://malakrobo_description/meshes/rplidar.dae" scale="0.001 0.001 0.001" />
-      </geometry>
-    </visual>
-    <inertial>
-      <mass value="1e-5" />
-      <origin xyz="0 0 0" rpy="1.5707 0 4.71"/>
-      <inertia ixx="0" ixy="0" ixz="0" iyy="0" iyz="0" izz="0" />
-    </inertial>
-  </link>
-  <joint name="sensor_base_joint" type="fixed">
-    <axis xyz="0 0 0" />
-    <origin xyz="0 0 0.23" rpy="0 0 3.14"/>
-    <parent link="base2"/>
-    <child link="sensor_base"/>
-  </joint>
-  <joint name="camera_joint" type="fixed">
-    <axis xyz="0 0 0" />
-    <origin xyz="-0.025 0 0.05" rpy="0 0 3.14"/>
-    <parent link="sensor_base"/>
-    <child link="camera"/>
-  </joint>
-  <joint name="rplidar_joint" type="fixed">
-    <axis xyz="0 1 0" />
-    <origin xyz="0 0 0.10" rpy="0 0 3.14"/>
-    <parent link="sensor_base"/>
-    <child link="laser"/>
-  </joint>
-  <joint name="base_joint" type="fixed">
-    <origin rpy="0 0 0" xyz="0 0 0"/>
-    <parent link="base_link"/>
-    <child link="base2"/>
-    <axis xyz="0.0 1.0 0.0"/>
-  </joint>
-  <joint name="base2_joint" type="fixed">
-    <origin rpy="0 0 0" xyz="0.15 0 0"/>
-    <parent link="base2"/>
-    <child link="base3"/>
-    <axis xyz="0.0 0.0 0.0"/>
-  </joint>
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
Commit message: Adding full autonomous operation for the large ball, needs tiny adjusting. Leftovers removed from the robot (old gripper). TODO: Translating autonomous operation to medium and small balls. Model needs to be trained once again as it does not recognize balls from some angles due to lights / shading. Finally, full autonomous program needs to be implemented (all of the ball autonomous operations will be translated to functions and then called together for the full sequence)

File: malakrobo_description/urdf/malakrobo.xacro (robot description, xacro)
@@ -66,49 +66,11 @@
             <origin rpy="0 0 0" xyz="0 0 0.1"/>
             <geometry>
+                <box size="0.02 0.25 0.07"/>
+            </geometry>
+        </visual>
+        <collision>
+            <origin rpy="0 0 0" xyz="0 0 0.07"/>
+            <geometry>
                 <box size="0.02 0.25 0.1"/>
-            </geometry>
-        </visual>
-        <collision>
-            <origin rpy="0 0 0" xyz="0 0 0.1"/>
-            <geometry>
-                <box size="0.02 0.25 0.1"/>
-            </geometry>
-        </collision>
-        <inertial>
-            <mass value="1"/>
-            <origin rpy="0 0 0" xyz="0 0 0"/>
-            <inertia ixx="1" ixy="0" ixz="0" iyy="1" iyz="0" izz="1"/>
-        </inertial>
-    </link>
-    <link name="left_fence">
-        <visual>
-            <origin rpy="1.0 1.57 1.57" xyz="0 0 0"/>
-            <geometry>
-                <box size="0.1 0.01 0.12"/>
-            </geometry>
-        </visual>
-        <collision>
-            <origin rpy="1.57 -1.0 1.57" xyz="0 0 0"/>
-            <geometry>
-                <box size="0.1 0.01 0.12"/>
-            </geometry>
-        </collision>
-        <inertial>
-            <mass value="1"/>
-            <origin rpy="0 0 0" xyz="0 0 0"/>
-            <inertia ixx="1" ixy="0" ixz="0" iyy="1" iyz="0" izz="1"/>
-        </inertial>
-    </link>
-    <link name="right_fence">
-        <visual>
-            <origin rpy="-1.0 1.57 1.57" xyz="0 0 0"/>
-            <geometry>
-                <box size="0.1 0.01 0.12"/>
-            </geometry>
-        </visual>
-        <collision>
-            <origin rpy="1.57 1.0 1.57" xyz="0 0 0"/>
-            <geometry>
-                <box size="0.1 0.01 0.12"/>
             </geometry>
         </collision>
@@ -441,16 +403,4 @@
         <limit effort="30" velocity="1.0" lower="0" upper="0"/>
     </joint>
-    <joint name="base_to_left_fence" type="fixed">
-        <origin rpy="0 0 0" xyz="0.055 0.15 0.1"/>
-        <parent link="base_fence"/>
-        <child link="left_fence"/>
-        <axis xyz="0.0 1.0 0.0"/>
-    </joint>
-    <joint name="base_to_right_fence" type="fixed">
-        <origin rpy="0 0 0" xyz="0.055 -0.15 0.1"/>
-        <parent link="base_fence"/>
-        <child link="right_fence"/>
-        <axis xyz="0.0 1.0 0.0"/>
-    </joint>
     <joint name="front_caster_base_joint" type="continuous">
         <origin rpy="0 0 0" xyz="0.15 0 0.08"/>

Commit message: Implementing autonomous recognition of ball position and navigation to the ball base on that position

File: malakrobo_description/urdf/malakrobo.xacro (robot description, xacro)
@@ -254,5 +254,5 @@
     <link name="camera">
         <collision>
-            <origin xyz="0 0 0" rpy="0 0 0.0"/>
+            <origin xyz="0 0 0" rpy="0 0.0 0.0"/>
             <geometry>
                 <box size="${cameraSize} ${cameraSize} ${cameraSize}"/>
